File: output/pcbs/revxl.kicad_pcb (KiCad board)
At the start: 2 copper layers, 304 x 113 mm, 229 parts

Commit message: Added Ergogen Screenshot
Parts:
- moved LED51 0.43 mm to (120.0, 136.0)
- moved _8 0.43 mm to (192.7, 152.5)
- moved S52 0.43 mm to (260.0, 132.5)
- moved _17 0.43 mm to (296.0, 110.7)
- moved D35 0.43 mm to (230.1, 79.6)
- moved D39 0.43 mm to (211.6, 79.5)
- moved D6 0.43 mm to (75.4, 92.6)
- moved RE1 0.43 mm to (172.0, 124.4)
- moved D27 0.43 mm to (267.1, 79.8)
- moved LED32 0.43 mm to (252.0, 57.4)
- moved LED61 0.43 mm to (307.0, 59.5)
- moved _1 0.43 mm to (52.0, 58.0)
- moved D26 0.43 mm to (270.9, 96.4)
- moved LED63 0.43 mm to (325.0, 110.5)
- moved S30 0.43 mm to (260.7, 95.4)
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